File: R4875G1_ESP32S3_CAN_Controller/R4875G1_ESP32S3_CAN_Controller.kicad_sch (KiCad schematic)
At the start: 0 parts

Commit message: Started with first schematic session
Other:
- added sheet CAN_RS485 (CAN_RS485.kicad_sch)
- added sheet ESP32_S3 (ESP32_S3.kicad_sch)
- added sheet Power managemnet (Power managemnet.kicad_sch)
Changed lines of the file:
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@@
 	(generator_version "9.0")
 	(paper "A4")
+	(sheet
+		(at 30.48 31.75)
+		(size 30.48 43.18)
+		(exclude_from_sim no)
+		(in_bom yes)
+		(on_board yes)
+		(dnp no)
+		(fields_autoplaced yes)
+		(stroke
+			(width 0.1524)
+			(type solid)
+		)
+		(fill
+			(color 0 0 0 0.0000)
+		)
+		(property "Sheetname" "ESP32_S3"
+			(at 30.48 31.0384 0)
+			(effects
+				(font
+					(size 1.27 1.27)
+				)
+				(justify left bottom)
+			)
+		)
+		(property "Sheetfile" "ESP32_S3.kicad_sch"
+			(at 30.48 75.5146 0)
+			(effects
+				(font
+					(size 1.27 1.27)
+				)
+				(justify left top)
+			)
+		)
+		(instances
+			(project "R4875G1_ESP32S3_CAN_Controller"
+				(path "/1fcf8bb1-5391-44f4-930a-289d1bf41e92"
+					(page "2")
+				)
+			)
+		)
+	)
+	(sheet
+		(at 30.48 94.742)
+		(size 30.48 43.434)
+		(exclude_from_sim no)
+		(in_bom yes)
+		(on_board yes)
+		(dnp no)
+		(fields_autoplaced yes)
+		(stroke
+			(width 0.1524)
+			(type solid)
+		)
+		(fill
+			(color 0 0 0 0.0000)
+		)
+		(property "Sheetname" "CAN_RS485"
+			(at 30.48 94.0304 0)
+			(effects
+				(font
+					(size 1.27 1.27)
+				)
+				(justify left bottom)
+			)
+		)
+		(property "Sheetfile" "CAN_RS485.kicad_sch"
+			(at 30.48 138.7606 0)
+			(effects
+				(font
+					(size 1.27 1.27)
+				)
+				(justify left top)
+			)
+		)
+		(instances
+			(project "R4875G1_ESP32S3_CAN_Controller"
+				(path "/1fcf8bb1-5391-44f4-930a-289d1bf41e92"
+					(page "4")
+				)
+			)
+		)
+	)
+	(sheet
+		(at 76.2 31.75)
+		(size 30.48 43.18)
+		(exclude_from_sim no)
+		(in_bom yes)
+		(on_board yes)
+		(dnp no)
+		(fields_autoplaced yes)
+		(stroke
+			(width 0.1524)
+			(type solid)
+		)
+		(fill
+			(color 0 0 0 0.0000)
+		)
+		(property "Sheetname" "Power managemnet"
+			(at 76.2 31.0384 0)
+			(effects
+				(font
+					(size 1.27 1.27)
+				)
+				(justify left bottom)
+			)
+		)
+		(property "Sheetfile" "Power managemnet.kicad_sch"
+			(at 76.2 75.5146 0)
+			(effects
+				(font
+					(size 1.27 1.27)
+				)
+				(justify left top)
+			)
+		)
+		(property "Field2" ""
+			(at 76.2 31.75 0)
+			(effects
+				(font
+					(size 1.27 1.27)
+				)
+			)
+		)
+		(property "Field3" ""
+			(at 76.2 31.75 0)
+			(effects
+				(font
+					(size 1.27 1.27)
+				)
+			)
+		)
+		(property "Field4" ""
+			(at 76.2 31.75 0)
+			(effects
+				(font
+					(size 1.27 1.27)
+				)
+			)
+		)
+		(property "Field5" ""
+			(at 76.2 31.75 0)
+			(effects
+				(font
+					(size 1.27 1.27)
+				)
+			)
+		)
+		(instances
+			(project "R4875G1_ESP32S3_CAN_Controller"
+				(path "/1fcf8bb1-5391-44f4-930a-289d1bf41e92"
+					(page "3")
+				)
+			)
+		)
+	)
 	(sheet_instances
 		(path "/"
