File: R4875G1_ESP32S3_CAN_Controller.kicad_sch (KiCad schematic)
At the start: 0 parts

Commit message: Added Kicad files
Other:
- added sheet Human interface_HI (HI.kicad_sch)
Changed lines of the file:
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@@
+		)
+	)
+	(sheet
+		(at 76.2 95.25)
+		(size 30.48 43.18)
+		(exclude_from_sim no)
+		(in_bom yes)
+		(on_board yes)
+		(dnp no)
+		(fields_autoplaced yes)
+		(stroke
+			(width 0.1524)
+			(type solid)
+		)
+		(fill
+			(color 0 0 0 0.0000)
+		)
+		(property "Sheetname" "Human interface_HI"
+			(at 76.2 94.5384 0)
+			(effects
+				(font
+					(size 1.27 1.27)
+				)
+				(justify left bottom)
+			)
+		)
+		(property "Sheetfile" "HI.kicad_sch"
+			(at 76.2 139.0146 0)
+			(effects
+				(font
+					(size 1.27 1.27)
+				)
+				(justify left top)
+			)
+		)
+		(instances
+			(project "R4875G1_ESP32S3_CAN_Controller"
+				(path "/1fcf8bb1-5391-44f4-930a-289d1bf41e92"
+					(page "5")
+				)
+			)
 		)
 	)
